File: source/application specific/LPF-A-v1/LPF-A-v1.kicad_sch (KiCad schematic)
At the start: 33 parts, among them J1 Conn_01x01_Pin, J2 Conn_01x01_Pin, J3 Conn_01x01_Pin, J4 Conn_01x01_Pin, J5 Conn_01x01_Pin, J6 Conn_01x01_Pin, J7 Conn_01x01_Pin, U1 OPA140, U2 OPA140

Commit message: Update LPF-A-v1.kicad_sch
Parts:
- C7, C8: value 47n -> 10n
- R7: value 1k -> 2.2k
- R8: value 100 -> 220
Other:
- note added: "1. Do not split & prefilter. 2. PCR very important."
- note removed: "Do not split & prefilter"
Changed lines of the file:
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@@
 		)
 	)
-	(text "Do not split\n& prefilter"
+	(text "1. Do not split & prefilter.\n2. PCR very important."
 		(exclude_from_sim no)
 		(at 74.93 70.485 0)
@@
 			)
 		)
-		(property "Value" "1k"
+		(property "Value" "2.2k"
 			(at 180.975 95.25 90)
 			(effects
@@
 			)
 		)
-		(property "Value" "100"
+		(property "Value" "220"
 			(at 180.975 80.01 90)
 			(effects
@@
 			)
 		)
-		(property "Value" "47n"
+		(property "Value" "10n"
 			(at 193.675 88.8999 0)
 			(effects
@@
 			)
 		)
-		(property "Value" "47n"
+		(property "Value" "10n"
 			(at 173.355 88.8999 0)
 			(effects

Commit message: Switched 0805 resistor to 1206
Parts:
- R1: footprint Resistor_SMD:R_0805_2012Metric_Pad1.20x1.40mm_HandSolder -> Resistor_SMD:R_1206_3216Metric_Pad1.30x1.75mm_HandSolder
Changed lines of the file:
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@@
 			)
 		)
-		(property "Footprint" "Resistor_SMD:R_0805_2012Metric_Pad1.20x1.40mm_HandSolder"
+		(property "Footprint" "Resistor_SMD:R_1206_3216Metric_Pad1.30x1.75mm_HandSolder"
 			(at 74.295 81.788 90)
 			(effects

Commit message: Added pad for external resistor input
Parts:
- added J8: Conn_01x01_Pin, Manhattan:Manhattan-2mm, symbol Connector:Conn_01x01_Pin
- R1: footprint Resistor_SMD:R_1206_3216Metric_Pad1.30x1.75mm_HandSolder -> Resistor_SMD:R_0805_2012Metric_Pad1.20x1.40mm_HandSolder
Connections:
- net Debug renamed InR
- net InR: now also J8.1 (Pin_1)
Changed lines of the file:
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@@
 	)
 	(junction
-		(at 140.97 80.01)
-		(diameter 0)
-		(color 0 0 0 0)
-	)
-	(junction
 		(at 102.235 111.76)
 		(diameter 0)
@@
 	(wire
 		(pts
-			(xy 140.97 80.01) (xy 142.875 80.01)
-		)
-		(stroke
-			(width 0)
-			(type default)
-		)
-	)
-	(wire
-		(pts
 			(xy 208.28 105.41) (xy 210.82 105.41)
 		)
@@
 	(wire
 		(pts
-			(xy 135.255 80.01) (xy 140.97 80.01)
+			(xy 135.255 80.01) (xy 142.875 80.01)
 		)
 		(stroke
@@
 	(wire
 		(pts
+			(xy 208.28 132.08) (xy 211.455 132.08)
+		)
+		(stroke
+			(width 0)
+			(type default)
+		)
+	)
+	(wire
+		(pts
 			(xy 92.075 111.76) (xy 102.235 111.76)
 		)
@@
 	(wire
 		(pts
+			(xy 69.215 62.23) (xy 92.075 62.23)
+		)
+		(stroke
+			(width 0)
+			(type default)
+		)
+	)
+	(wire
+		(pts
 			(xy 189.865 118.11) (xy 189.865 119.38)
 		)
@@
 	(wire
 		(pts
-			(xy 140.97 67.945) (xy 140.97 80.01)
+			(xy 159.385 73.66) (xy 158.115 73.66)
 		)
 		(stroke
@@
 	(wire
 		(pts
-			(xy 159.385 73.66) (xy 158.115 73.66)
+			(xy 109.855 111.76) (xy 109.855 113.03)
 		)
 		(stroke
@@
 	(wire
 		(pts
-			(xy 109.855 111.76) (xy 109.855 113.03)
+			(xy 146.685 118.11) (xy 147.955 118.11)
 		)
 		(stroke
@@
 	(wire
 		(pts
-			(xy 146.685 118.11) (xy 147.955 118.11)
+			(xy 84.455 80.01) (xy 92.075 80.01)
 		)
 		(stroke
@@
 	(wire
 		(pts
-			(xy 84.455 80.01) (xy 92.075 80.01)
+			(xy 92.075 62.23) (xy 92.075 80.01)
 		)
 		(stroke
@@
 	(wire
 		(pts
-			(xy 140.97 67.945) (xy 154.305 67.945)
-		)
-		(stroke
-			(width 0)
-			(type default)
-		)
-	)
-	(wire
-		(pts
 			(xy 209.55 124.46) (xy 209.55 125.095)
 		)
@@
 		)
 	)
-	(global_label "Debug"
-		(shape input)
-		(at 154.305 67.945 0)
-		(fields_autoplaced yes)
-		(effects
-			(font
-				(size 1.27 1.27)
-			)
-			(justify left)
-		)
-		(property "Intersheetrefs" "${INTERSHEET_REFS}"
-			(at 163.0958 67.945 0)
-			(effects
-				(font
-					(size 1.27 1.27)
-				)
-				(justify left)
-				(hide yes)
-			)
-		)
-	)
 	(global_label "Out"
 		(shape input)
@@
 		)
 	)
+	(global_label "InR"
+		(shape input)
+		(at 211.455 132.08 0)
+		(fields_autoplaced yes)
+		(effects
+			(font
+				(size 1.27 1.27)
+			)
+			(justify left)
+		)
+		(property "Intersheetrefs" "${INTERSHEET_REFS}"
+			(at 217.464 132.08 0)
+			(effects
+				(font
+					(size 1.27 1.27)
+				)
+				(justify left)
+				(hide yes)
+			)
+		)
+	)
 	(global_label "U2 V+"
 		(shape input)
@@
 		)
 	)
+	(global_label "InR"
+		(shape input)
+		(at 69.215 62.23 180)
+		(fields_autoplaced yes)
+		(effects
+			(font
+				(size 1.27 1.27)
+			)
+			(justify right)
+		)
+		(property "Intersheetrefs" "${INTERSHEET_REFS}"
+			(at 63.206 62.23 0)
+			(effects
+				(font
+					(size 1.27 1.27)
+				)
+				(justify right)
+				(hide yes)
+			)
+		)
+	)
 	(symbol
 		(lib_id "Device:R")
@@
 			)
 		)
-		(property "Footprint" "Resistor_SMD:R_1206_3216Metric_Pad1.30x1.75mm_HandSolder"
+		(property "Footprint" "Resistor_SMD:R_0805_2012Metric_Pad1.20x1.40mm_HandSolder"
 			(at 74.295 81.788 90)
 			(effects
@@
 					(unit 1)
 				)
+			)
+		)
+	)
+	(symbol
+		(lib_id "Connector:Conn_01x01_Pin")
+		(at 203.2 132.08 0)
+		(unit 1)
+		(exclude_from_sim no)
+		(in_bom yes)
+		(on_board yes)
+		(dnp no)
+		(property "Reference" "J8"
+			(at 201.168 132.08 0)
+			(effects
+				(font
+					(size 1.27 1.27)
+				)
+			)
+		)
+		(property "Value" "Conn_01x01_Pin"
+			(at 203.835 129.54 0)
+			(effects
+				(font
+					(size 1.27 1.27)
+				)
+				(hide yes)
+			)
+		)
+		(property "Footprint" "Manhattan:Manhattan-2mm"
+			(at 203.2 132.08 0)
+			(effects
+				(font
+					(size 1.27 1.27)
+				)
+				(hide yes)
+			)
+		)
+		(property "Datasheet" "~"
+			(at 203.2 132.08 0)
+			(effects
+				(font
+					(size 1.27 1.27)
+				)
+				(hide yes)
+			)
+		)
+		(property "Description" "Generic connector, single row, 01x01, script generated"
+			(at 203.2 132.08 0)
+			(effects
+				(font
+					(size 1.27 1.27)
+				)
+				(hide yes)
+			)
+		)
+		(pin "1"
+		)
+		(instances
+			(project "LPF-A-v1"
+				(path "/d3145d82-6a37-4f1e-9453-e65b2855fcb5"
+					(reference "J8")
+					(unit 1)
+				)

Commit message: Updated output capacitors to 0805
Parts:
- C7, C8: footprint Resistor_SMD:R_0603_1608Metric_Pad0.98x0.95mm_HandSolder -> Resistor_SMD:R_0805_2012Metric_Pad1.20x1.40mm_HandSolder
Changed lines of the file:
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@@
 			)
 		)
-		(property "Footprint" "Resistor_SMD:R_0603_1608Metric_Pad0.98x0.95mm_HandSolder"
+		(property "Footprint" "Resistor_SMD:R_0805_2012Metric_Pad1.20x1.40mm_HandSolder"
 			(at 190.8302 91.44 0)
 			(effects
@@
 			)
 		)
-		(property "Footprint" "Resistor_SMD:R_0603_1608Metric_Pad0.98x0.95mm_HandSolder"
+		(property "Footprint" "Resistor_SMD:R_0805_2012Metric_Pad1.20x1.40mm_HandSolder"
 			(at 170.5102 91.44 0)
 			(effects

Commit message: Added pad to allow for external sense
Parts:
- added J9: Conn_01x01_Pin, Manhattan:Manhattan-2mm, symbol Connector:Conn_01x01_Pin
- added R13: 2.2k, Resistor_SMD:R_0603_1608Metric_Pad0.98x0.95mm_HandSolder, symbol Device:R
Connections:
- net at C7.2, R7.1, U2.2 (-): now also R13.1
- new net OutSense: J9.1 (Pin_1), R13.2
Other:
- note added: "Populate R7 or R13, depending on internal or external sense"
- moved on the sheet: C10, C11, C12, C9, J1, J2, J3, J4, J5, J6, J7, J8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
