File: source/application specific/ADC-B-v1/ADC-B-v1.kicad_pcb (KiCad board)
At the start: 4 copper layers, 20.5 x 10.5 mm, 22 parts, among them U1 AD7276, U2 OPA354

Commit message: Updated ADC-B-v1
Parts:
- removed C4: 10μF, Capacitor_Tantalum_SMD:CP_EIA-2012-15_AVX-P
- removed FB1: FerriteBead_Small, Resistor_SMD:R_0603_1608Metric_Pad0.98x0.95mm_HandSolder
- C1: value 680nF -> 100nF; footprint Capacitor_SMD:C_0402_1005Metric_Pad0.74x0.62mm_HandSolder -> Capacitor_SMD:C_0603_1608Metric_Pad1.08x0.95mm_HandSolder
- C3: value 100nF -> 10μF; footprint Capacitor_SMD:C_0402_1005Metric_Pad0.74x0.62mm_HandSolder -> Capacitor_SMD:C_1206_3216Metric_Pad1.33x1.80mm_HandSolder
- C6: footprint Capacitor_SMD:C_0402_1005Metric_Pad0.74x0.62mm_HandSolder -> Capacitor_SMD:C_0603_1608Metric_Pad1.08x0.95mm_HandSolder
- R4, R5, R6: footprint Resistor_SMD:R_0402_1005Metric -> Resistor_SMD:R_0603_1608Metric_Pad0.98x0.95mm_HandSolder
- moved C3 3.20 mm to (147.5, 96.2), turned to 180 degrees
- moved C6 1.46 mm to (151.2, 103.0), turned to 180 degrees
- moved R6 0.96 mm to (151.2, 100.2)
- moved R5 0.87 mm to (151.2, 99.1)
- moved R4 0.81 mm to (151.2, 98.0)
- moved R2 0.75 mm to (151.2, 101.8)
- moved C1 0.41 mm to (144.4, 98.1)
- moved U1 0.38 mm to (147.5, 99.1)
- moved C2 0.20 mm to (142.9, 99.6)
- moved R1 0.12 mm to (144.4, 101.1)
Connections:
- C1 pad 2: Net-(U1-VDD) -> +3.3V
- C3 pad 2: Net-(U1-VDD) -> +3.3V
- U1 pad 1: Net-(U1-VDD) -> +3.3V
Routing:
- net /IN: track 6.37 -> 4.15 mm, vias 2 -> 0
- net /SCK: track 5.92 -> 4.66 mm
- net GND: track 0.00 -> 1.12 mm, vias 4 -> 5
- net /~{CS}: track 5.92 -> 4.97 mm
- net /SDO: track 5.28 -> 4.41 mm
- net +3.3V: track 0.85 -> 1.50 mm
- net Net-(U1-~{CS}): track 1.32 -> 1.95 mm
- net Net-(U1-SCK): track 1.32 -> 1.95 mm
- net Net-(U2-V+): track 2.46 -> 3.03 mm
- net Net-(U1-SDO): track 1.32 -> 1.88 mm
- removed copper zone on F.Cu, net Net-(U1-VDD)
Other:
- board text added: "BF"
- board text removed: "OA"
