File: source/application specific/ADC-B-v1/ADC-B-v1.kicad_sch (KiCad schematic)
At the start: 22 parts, among them U1 AD7276, U2 OPA354

Commit message: Updated ADC-B-v1
Parts:
- removed C4: 10μF, Capacitor_Tantalum_SMD:CP_EIA-2012-15_AVX-P, symbol Device:C_Polarized_Small
- removed FB1: FerriteBead_Small, Resistor_SMD:R_0603_1608Metric_Pad0.98x0.95mm_HandSolder, symbol Device:FerriteBead_Small
- C1: value 680nF -> 100nF; footprint Capacitor_SMD:C_0402_1005Metric_Pad0.74x0.62mm_HandSolder -> Capacitor_SMD:C_0603_1608Metric_Pad1.08x0.95mm_HandSolder
- C3: value 100nF -> 10μF; footprint Capacitor_SMD:C_0402_1005Metric_Pad0.74x0.62mm_HandSolder -> Capacitor_SMD:C_1206_3216Metric_Pad1.33x1.80mm_HandSolder
- C6: footprint Capacitor_SMD:C_0402_1005Metric_Pad0.74x0.62mm_HandSolder -> Capacitor_SMD:C_0603_1608Metric_Pad1.08x0.95mm_HandSolder
- R4, R5, R6: footprint Resistor_SMD:R_0402_1005Metric -> Resistor_SMD:R_0603_1608Metric_Pad0.98x0.95mm_HandSolder
Connections:
- net +3.3V: now also C1.2, C3.2, U1.1 (VDD)
Other:
- note removed: "Datasheet recommends 1μF tantalum in parallel with 100nF ceramic, 680nF ceramic also placed close to reference pin"
- note removed: "Ferrite or low value resistor"
Changed lines of the file:
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@@
 	(paper "A4")
-	(junction
-		(at 142.24 80.01)
-		(diameter 0)
-		(color 0 0 0 0)
-	)
 	(junction
 		(at 129.54 101.6)
@@
 	)
 	(junction
-		(at 152.4 69.85)
-		(diameter 0)
-		(color 0 0 0 0)
-	)
-	(junction
 		(at 116.84 91.44)
 		(diameter 0)
@@
 	(wire
 		(pts
-			(xy 152.4 69.85) (xy 152.4 80.01)
+			(xy 152.4 74.93) (xy 152.4 80.01)
 		)
 		(stroke
@@
 	(wire
 		(pts
-			(xy 152.4 64.77) (xy 152.4 69.85)
-		)
-		(stroke
-			(width 0)
-			(type default)
-		)
-	)
-	(wire
-		(pts
 			(xy 236.22 101.6) (xy 241.3 101.6)
 		)
@@
 	(wire
 		(pts
-			(xy 149.86 69.85) (xy 152.4 69.85)
-		)
-		(stroke
-			(width 0)
-			(type default)
-		)
-	)
-	(wire
-		(pts
 			(xy 116.84 76.2) (xy 116.84 78.74)
 		)
@@
 	(wire
 		(pts
-			(xy 142.24 69.85) (xy 144.78 69.85)
-		)
-		(stroke
-			(width 0)
-			(type default)
-		)
-	)
-	(wire
-		(pts
 			(xy 116.84 91.44) (xy 116.84 93.98)
 		)
@@
 			(width 0)
 			(type default)
-		)
-	)
-	(wire
-		(pts
-			(xy 152.4 57.15) (xy 152.4 59.69)
-		)
-		(stroke
-			(width 0)
-			(type default)
-		)
-	)
-	(wire
-		(pts
-			(xy 142.24 69.85) (xy 142.24 80.01)
-		)
-		(stroke
-			(width 0)
-			(type default)
-		)
-	)
-	(text "Datasheet recommends 1μF tantalum\nin parallel with 100nF ceramic, 680nF \nceramic also placed close to\nreference pin"
-		(exclude_from_sim no)
-		(at 156.21 76.835 0)
-		(effects
-			(font
-				(size 1.27 1.27)
-			)
-			(justify left top)
-		)
-	)
-	(text "Ferrite or low value resistor"
-		(exclude_from_sim no)
-		(at 168.275 66.675 0)
-		(effects
-			(font
-				(size 1.27 1.27)
-			)
 		)
 	)
@@
 			)
 		)
-		(property "Footprint" "Resistor_SMD:R_0402_1005Metric"
+		(property "Footprint" "Resistor_SMD:R_0603_1608Metric_Pad0.98x0.95mm_HandSolder"
 			(at 166.37 100.838 90)
 			(effects
@@
 			)
 		)
-		(property "Value" "680nF"
+		(property "Value" "100nF"
 			(at 147.3263 86.36 90)
 			(effects
@@
 			)
 		)
-		(property "Footprint" "Capacitor_SMD:C_0402_1005Metric_Pad0.74x0.62mm_HandSolder"
+		(property "Footprint" "Capacitor_SMD:C_0603_1608Metric_Pad1.08x0.95mm_HandSolder"
 			(at 147.32 90.17 0)
 			(effects
@@
 	)
 	(symbol
-		(lib_id "Device:FerriteBead_Small")
-		(at 152.4 62.23 0)
-		(unit 1)
-		(exclude_from_sim no)
-		(in_bom yes)
-		(on_board yes)
-		(dnp no)
-		(fields_autoplaced yes)
-		(property "Reference" "FB1"
-			(at 154.94 60.9218 0)
-			(effects
-				(font
-					(size 1.27 1.27)
-				)
-				(justify left)
-			)
-		)
-		(property "Value" "FerriteBead_Small"
-			(at 154.94 63.4618 0)
-			(effects
-				(font
-					(size 1.27 1.27)
-				)
-				(justify left)
-			)
-		)
-		(property "Footprint" "Resistor_SMD:R_0603_1608Metric_Pad0.98x0.95mm_HandSolder"
-			(at 150.622 62.23 90)
-			(effects
-				(font
-					(size 1.27 1.27)
-				)
-				(hide yes)
-			)
-		)
-		(property "Datasheet" "~"
-			(at 152.4 62.23 0)
-			(effects
-				(font
-					(size 1.27 1.27)
-				)
-				(hide yes)
-			)
-		)
-		(property "Description" "Ferrite bead, small symbol"
-			(at 152.4 62.23 0)
-			(effects
-				(font
-					(size 1.27 1.27)
-				)
-				(hide yes)
-			)
-		)
-		(pin "1"
-		)
-		(pin "2"
-		)
-		(instances
-			(project "ADC-B-v1"
-				(path "/504ec218-cb88-462b-a811-05e6cf14a2b1"
-					(reference "FB1")
-					(unit 1)
-				)
-			)
-		)
-	)
-	(symbol
 		(lib_id "power:GND")
 		(at 238.76 69.85 270)
@@
 			)
 		)
-		(property "Value" "100nF"
+		(property "Value" "10μF"
 			(at 147.3263 76.2 90)
 			(effects
@@
 			)
 		)
-		(property "Footprint" "Capacitor_SMD:C_0402_1005Metric_Pad0.74x0.62mm_HandSolder"
+		(property "Footprint" "Capacitor_SMD:C_1206_3216Metric_Pad1.33x1.80mm_HandSolder"
 			(at 147.32 80.01 0)
 			(effects
@@
 	(symbol
 		(lib_id "power:+3.3V")
-		(at 152.4 57.15 0)
+		(at 152.4 74.93 0)
 		(unit 1)
 		(exclude_from_sim no)
@@
 		(fields_autoplaced yes)
 		(property "Reference" "#PWR03"
-			(at 152.4 60.96 0)
+			(at 152.4 78.74 0)
 			(effects
 				(font
@@
 		)
 		(property "Value" "+3.3V"
-			(at 152.4 52.07 0)
+			(at 152.4 69.85 0)
 			(effects
 				(font
@@
 		)
 		(property "Footprint" ""
-			(at 152.4 57.15 0)
+			(at 152.4 74.93 0)
 			(effects
 				(font
@@
 		)
 		(property "Datasheet" ""
-			(at 152.4 57.15 0)
+			(at 152.4 74.93 0)
 			(effects
 				(font
@@
 		)
 		(property "Description" "Power symbol creates a global label with name \"+3.3V\""
-			(at 152.4 57.15 0)
+			(at 152.4 74.93 0)
 			(effects
 				(font
@@
 			)
 		)
-		(property "Footprint" "Resistor_SMD:R_0402_1005Metric"
+		(property "Footprint" "Resistor_SMD:R_0603_1608Metric_Pad0.98x0.95mm_HandSolder"
 			(at 186.69 105.918 90)
 			(effects
@@
 	)
 	(symbol
-		(lib_id "Device:C_Polarized_Small")
-		(at 147.32 69.85 270)
-		(unit 1)
-		(exclude_from_sim no)
-		(in_bom yes)
-		(on_board yes)
-		(dnp no)
-		(fields_autoplaced yes)
-		(property "Reference" "C4"
-			(at 147.8661 63.5 90)
-			(effects
-				(font
-					(size 1.27 1.27)
-				)
-			)
-		)
-		(property "Value" "10μF"
-			(at 147.8661 66.04 90)
-			(effects
-				(font
-					(size 1.27 1.27)
-				)
-			)
-		)
-		(property "Footprint" "Capacitor_Tantalum_SMD:CP_EIA-2012-15_AVX-P"
-			(at 147.32 69.85 0)
-			(effects
-				(font
-					(size 1.27 1.27)
-				)
-				(hide yes)
-			)
-		)
-		(property "Datasheet" "~"
-			(at 147.32 69.85 0)
-			(effects
-				(font
-					(size 1.27 1.27)
-				)
-				(hide yes)
-			)
-		)
-		(property "Description" "Polarized capacitor, small symbol"
-			(at 147.32 69.85 0)
-			(effects
-				(font
-					(size 1.27 1.27)
-				)
-				(hide yes)
-			)
-		)
-		(pin "2"
-		)
-		(pin "1"
-		)
-		(instances
-			(project "ADC-B-v1"
-				(path "/504ec218-cb88-462b-a811-05e6cf14a2b1"
-					(reference "C4")
-					(unit 1)
-				)
-			)
-		)
-	)
-	(symbol
 		(lib_id "Connector:TestPoint")
 		(at 241.3 88.9 270)
@@
 			)
 		)
-		(property "Footprint" "Capacitor_SMD:C_0402_1005Metric_Pad0.74x0.62mm_HandSolder"
+		(property "Footprint" "Capacitor_SMD:C_0603_1608Metric_Pad1.08x0.95mm_HandSolder"
 			(at 111.76 91.44 0)
 			(effects
@@
 			)
 		)
-		(property "Footprint" "Resistor_SMD:R_0402_1005Metric"
+		(property "Footprint" "Resistor_SMD:R_0603_1608Metric_Pad0.98x0.95mm_HandSolder"
 			(at 176.53 103.378 90)
 			(effects
